File: hardware/pump/pump.kicad_pcb (KiCad board)
At the start: 2 copper layers, 50.8 x 36.8 mm, 14 parts, among them J1 DB9_Male, J2 PumpThermocoupleAdc, J3 GroupheadThermistor, J4 PumpConnect, J5 HeaterRelayConnect, K1 G3MC202PDC5

Commit message: Add label, adjust ground plane
Other:
- board text added: "GH_TEMP"
